Commit message: Update BRUCE URDF version to 0.0.6 and fix joint orders for hip roll and pitch

File: Gazebo/models/bruce/urdf/bruce.urdf (robot description, URDF)
Before this commit: robot bruce, 17 links, 16 joints
Links:
- link hip_pitch_link_l: mass 0.72062828 -> 0.05; geometry collision mesh filename=package://bruce/meshes/hip_roll_link_l.STL; visual mesh filename=package://bruce/meshes/hip_roll_link_l.STL
- link hip_pitch_link_r: mass 0.72848988 -> 0.05; geometry collision mesh filename=package://bruce/meshes/hip_roll_link_r.STL; visual mesh filename=package://bruce/meshes/hip_roll_link_r.STL
- link hip_roll_link_l: mass 0.05 -> 0.72062828; geometry collision mesh filename=package://bruce/meshes/hip_pitch_link_l.STL; visual mesh filename=package://bruce/meshes/hip_pitch_link_l.STL
- link hip_roll_link_r: mass 0.05 -> 0.72848988; geometry collision mesh filename=package://bruce/meshes/hip_pitch_link_r.STL; visual mesh filename=package://bruce/meshes/hip_pitch_link_r.STL
Joints:
- joint hip_pitch_l: axis 0 0 1 -> 0 -1 0; origin xyz=0 0 0 rpy=1.570796327 0 0 -> xyz=0 0 0 rpy=1.570796327 1.570796327 3.14159; parent hip_roll_link_l -> hip_yaw_link_l
- joint hip_pitch_r: axis 0 0 1 -> 0 -1 0; origin xyz=0 0 0 rpy=1.570796327 0 0 -> xyz=0 0 0 rpy=-1.570796327 1.570796327 0; parent hip_roll_link_r -> hip_yaw_link_r
- joint hip_roll_l: axis 0 0 1 -> 0 -1 0; origin xyz=0 0 0 rpy=1.570796327 1.570796327 3.14159 -> xyz=0 0 0 rpy=1.570796327 0 0; parent hip_yaw_link_l -> hip_pitch_link_l
- joint hip_roll_r: axis 0 0 1 -> 0 -1 0; origin xyz=0 0 0 rpy=-1.570796327 1.570796327 0 -> xyz=0 0 0 rpy=1.570796327 0 0; parent hip_yaw_link_r -> hip_pitch_link_r
- joint knee_pitch_l: parent hip_pitch_link_l -> hip_roll_link_l
- joint knee_pitch_r: parent hip_pitch_link_r -> hip_roll_link_r
