Commit message: Delete empty joints and links in urdf.

File: Gazebo/urdf/bruce.urdf (robot description, URDF)
Before this commit: robot bruce, 18 links, 16 joints
Links:
- removed link 

Commit message: Update mass and intertia

File: Gazebo/urdf/bruce.urdf (robot description, URDF)
Before this commit: robot bruce, 17 links, 16 joints
Links:
- link hip_pitch_link_l: mass 0.72062828 -> 0.0129553
- link hip_pitch_link_r: mass 0.72848988 -> 0.0129553
- link hip_roll_link_l: mass 0.05 -> 0.66351862
- link hip_roll_link_r: mass 0.05 -> 0.66351862
